File: Teensy-Field-XLR.kicad_sch (KiCad schematic)
At the start: 0 parts

Commit message: schematic
Parts:
- added U1: Teensy4.1, jannett_footprints:Teensy41, symbol jannett_symbols:Teensy4.1
- added U2: PCM1860DBT, Package_SO:TSSOP-30_4.4x7.8mm_P0.5mm, symbol Audio:PCM1860DBT
Connections:
- new net +3.3V: U1.15 (3V3), U1.46 (3V3), U1.51 (3V3)
- new net GND: U1.1 (GND), U1.34 (GND), U1.47 (GND), U1.52 (GND), U2.12 (DGND), U2.7 (AGND)
